File: hardware/onoffschim.kicad_sch (KiCad schematic)
At the start: 9 parts, among them Q7 AO3401A, Q8 2N7002

Commit message: Add BOM descriptions and JLC PCB LCSC part numbers. Generate gerber, drill and pick-and-place files.
Parts:
- C21: Comment (none) -> X5R 16V; LCSC (none) -> EMK107ABJ475KA-T
- D1: Comment (none) -> 30V; LCSC (none) -> C134405
- Q7: Comment (none) -> 30V; LCSC (none) -> C306862
- Q8: Comment (none) -> 60V; LCSC (none) -> C350313
- R24, R25, R26, R27, R28: Comment (none) -> 5% 100ppm
Changed lines of the file:
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@@
+      (effects (font (size 1.27 1.27)) hide)
+    )
+    (property "Comment" "5% 100ppm" (id 4) (at 135.89 101.6 0)
       (effects (font (size 1.27 1.27)) hide)
     )
@@
       (effects (font (size 1.27 1.27)) hide)
     )
+    (property "Comment" "5% 100ppm" (id 4) (at 157.48 67.31 0)
+      (effects (font (size 1.27 1.27)) hide)
+    )
     (pin "1")
     (pin "2")
@@
     )
     (property "Datasheet" "~" (id 3) (at 135.89 111.76 0)
+      (effects (font (size 1.27 1.27)) hide)
+    )
+    (property "Comment" "X5R 16V" (id 4) (at 135.89 111.76 0)
+      (effects (font (size 1.27 1.27)) hide)
+    )
+    (property "LCSC" "EMK107ABJ475KA-T" (id 5) (at 135.89 111.76 0)
       (effects (font (size 1.27 1.27)) hide)
     )
@@
       (effects (font (size 1.27 1.27)) (justify left) hide)
     )
+    (property "Comment" "60V" (id 4) (at 119.38 106.68 0)
+      (effects (font (size 1.27 1.27)) hide)
+    )
+    (property "LCSC" "C350313" (id 5) (at 119.38 106.68 0)
+      (effects (font (size 1.27 1.27)) hide)
+    )
     (pin "1")
     (pin "2")
@@
       (effects (font (size 1.27 1.27)) hide)
     )
+    (property "Comment" "5% 100ppm" (id 4) (at 104.14 73.66 0)
+      (effects (font (size 1.27 1.27)) hide)
+    )
     (pin "1")
     (pin "2")
@@
     (property "Datasheet" "http://www.aosmd.com/pdfs/datasheet/AO3401A.pdf" (id 3) (at 116.84 64.77 0)
       (effects (font (size 1.27 1.27)) (justify left) hide)
+    )
+    (property "Comment" "30V" (id 4) (at 116.84 64.77 0)
+      (effects (font (size 1.27 1.27)) hide)
+    )
+    (property "LCSC" "C306862" (id 5) (at 116.84 64.77 0)
+      (effects (font (size 1.27 1.27)) hide)
     )
     (pin "1")
@@
     )
     (property "Datasheet" "~" (id 3) (at 135.89 67.31 0)
+      (effects (font (size 1.27 1.27)) hide)
+    )
+    (property "Comment" "5% 100ppm" (id 4) (at 135.89 67.31 0)
       (effects (font (size 1.27 1.27)) hide)
     )
@@
       (effects (font (size 1.27 1.27)) hide)
     )
+    (property "Comment" "5% 100ppm" (id 4) (at 125.73 83.82 0)
+      (effects (font (size 1.27 1.27)) hide)
+    )
     (pin "1")
     (pin "2")
@@
       (effects (font (size 1.27 1.27)) hide)
     )
+    (property "Comment" "30V" (id 4) (at 147.32 74.93 0)
+      (effects (font (size 1.27 1.27)) hide)
+    )
+    (property "LCSC" "C134405" (id 5) (at 147.32 74.93 0)
+      (effects (font (size 1.27 1.27)) hide)
+    )

Commit message: Smaller high value caps. Standard R/C footprints instead of hand solder.
Parts:
- C21: footprint Capacitor_SMD:C_0603_1608Metric_Pad1.08x0.95mm_HandSolder -> Capacitor_SMD:C_0603_1608Metric; Comment X5R 16V -> X7R 10V; LCSC EMK107ABJ475KA-T -> (none)
- D1: LCSC C134405 -> C37704
- Q7: LCSC C306862 -> C15127
- R24, R25, R26, R27, R28: footprint Resistor_SMD:R_0603_1608Metric_Pad0.98x0.95mm_HandSolder -> Resistor_SMD:R_0603_1608Metric
Changed lines of the file:
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@@
       (effects (font (size 1.27 1.27)) (justify right))
     )
-    (property "Footprint" "Resistor_SMD:R_0603_1608Metric_Pad0.98x0.95mm_HandSolder" (id 2) (at 137.668 101.6 90)
+    (property "Footprint" "Resistor_SMD:R_0603_1608Metric" (id 2) (at 137.668 101.6 90)
       (effects (font (size 1.27 1.27)) hide)
     )
@@
       (effects (font (size 1.27 1.27)) (justify right))
     )
-    (property "Footprint" "Resistor_SMD:R_0603_1608Metric_Pad0.98x0.95mm_HandSolder" (id 2) (at 159.258 67.31 90)
+    (property "Footprint" "Resistor_SMD:R_0603_1608Metric" (id 2) (at 159.258 67.31 90)
       (effects (font (size 1.27 1.27)) hide)
     )
@@
       (effects (font (size 1.27 1.27)) (justify left))
     )
-    (property "Footprint" "Capacitor_SMD:C_0603_1608Metric_Pad1.08x0.95mm_HandSolder" (id 2) (at 136.8552 115.57 0)
+    (property "Footprint" "Capacitor_SMD:C_0603_1608Metric" (id 2) (at 136.8552 115.57 0)
       (effects (font (size 1.27 1.27)) hide)
     )
@@
       (effects (font (size 1.27 1.27)) hide)
     )
-    (property "Comment" "X5R 16V" (id 4) (at 135.89 111.76 0)
-      (effects (font (size 1.27 1.27)) hide)
-    )
-    (property "LCSC" "EMK107ABJ475KA-T" (id 5) (at 135.89 111.76 0)
+    (property "Comment" "X7R 10V" (id 4) (at 135.89 111.76 0)
+      (effects (font (size 1.27 1.27)) hide)
+    )
+    (property "LCSC" "" (id 5) (at 135.89 111.76 0)
       (effects (font (size 1.27 1.27)) hide)
     )
@@
       (effects (font (size 1.27 1.27)) (justify right))
     )
-    (property "Footprint" "Resistor_SMD:R_0603_1608Metric_Pad0.98x0.95mm_HandSolder" (id 2) (at 105.918 73.66 90)
+    (property "Footprint" "Resistor_SMD:R_0603_1608Metric" (id 2) (at 105.918 73.66 90)
       (effects (font (size 1.27 1.27)) hide)
     )
@@
       (effects (font (size 1.27 1.27)) hide)
     )
-    (property "LCSC" "C306862" (id 5) (at 116.84 64.77 0)
+    (property "LCSC" " C15127" (id 5) (at 116.84 64.77 0)
       (effects (font (size 1.27 1.27)) hide)
     )
@@
       (effects (font (size 1.27 1.27)) (justify right))
     )
-    (property "Footprint" "Resistor_SMD:R_0603_1608Metric_Pad0.98x0.95mm_HandSolder" (id 2) (at 137.668 67.31 90)
+    (property "Footprint" "Resistor_SMD:R_0603_1608Metric" (id 2) (at 137.668 67.31 90)
       (effects (font (size 1.27 1.27)) hide)
     )
@@
     (property "Reference" "R25" (id 0) (at 125.73 77.47 90))
     (property "Value" "10k" (id 1) (at 125.73 80.01 90))
-    (property "Footprint" "Resistor_SMD:R_0603_1608Metric_Pad0.98x0.95mm_HandSolder" (id 2) (at 125.73 82.042 90)
+    (property "Footprint" "Resistor_SMD:R_0603_1608Metric" (id 2) (at 125.73 82.042 90)
       (effects (font (size 1.27 1.27)) hide)
     )
@@
       (effects (font (size 1.27 1.27)) hide)
     )
-    (property "LCSC" "C134405" (id 5) (at 147.32 74.93 0)
-      (effects (font (size 1.27 1.27)) hide)
-    )
+    (property "LCSC" "C37704" (id 5) (at 147.32 74.93 0)
+      (effects (font (size 1.27 1.27)) hide)
+    )
